File: CentralAvionicsHub.kicad_pcb (KiCad board)
At the start: 2 copper layers, 106.4 x 87.9 mm, 23 parts, among them J1 GPS/ARINC, J2 MFD, J3 PFD, J4 NavCom, J5 Airframe, J6 GND1, J7 GND2, J8 Power_In, J9 Switches_Indicators

Commit message: Replaced F1 footprint with traditional fuseholder for Mini Blade Fuse.
Changed R1-R5 to 1206

Modified footprint of DA15 to match TE part

Managed Libraries, regenerated gerbers at V1.
Parts:
- F1: footprint Fuse:Fuse_0805_2012Metric -> fuse_holder:FUSE_3568
- J8: footprint Connector_Dsub:DSUB-15_Socket_Vertical_P2.77x2.84mm_MountingHoles -> TE_DSUB:5787683 15 Pin Female Vertical
- R1, R2, R3, R4, R5: footprint Resistor_SMD:R_0805_2012Metric -> Resistor_SMD:R_1206_3216Metric_Pad1.30x1.75mm_HandSolder
- moved F1 17.5 mm to (115.8, 74.6), turned to -90 degrees
- moved J6 3.49 mm to (108.7, 66.9), turned to 90 degrees
- moved J7 1.10 mm to (123.3, 66.9), turned to 90 degrees
- moved J8 0.11 mm to (152.0, 70.1)
- moved R5 0.10 mm to (189.5, 143.7)
Routing:
- net Net-(J7-Pin_1): track 8.55 -> 0.29 mm
- net /Annunciator_V+: track 115.1 -> 111.9 mm
- net /GPS_V+: track 70.6 -> 73.4 mm
- net Net-(J9-Pad37): track 23.7 -> 23.1 mm
- net Net-(J9-Pad18): track 20.5 -> 19.8 mm
- net Net-(J9-Pad17): track 25.3 -> 24.7 mm
- net Net-(J9-Pad36): track 20.4 -> 19.7 mm
- net GND: vias 141 -> 145
Other:
- board text added: "Central Avionics Hub Rev 1: 24 November 2025"
- board text removed: "Central Avionics Hub Rev 0: 23 November 2025"
