File: CentralAvionicsHub.kicad_sch (KiCad schematic)
At the start: 22 parts, among them J1 GPS/ARINC, J2 MFD, J3 PFD, J4 NavCom, J5 Airframe, J6 GND1, J7 GND2, J8 Power_In, J9 Switches_Indicators

Commit message: Replaced F1 footprint with traditional fuseholder for Mini Blade Fuse.
Changed R1-R5 to 1206

Modified footprint of DA15 to match TE part

Managed Libraries, regenerated gerbers at V1.
Parts:
- F1: footprint Fuse:Fuse_0805_2012Metric -> fuse_holder:FUSE_3568
- J8: footprint Connector_Dsub:DSUB-15_Socket_Vertical_P2.77x2.84mm_MountingHoles -> TE_DSUB:5787683 15 Pin Female Vertical
- R1, R2, R3, R4, R5: footprint Resistor_SMD:R_0805_2012Metric -> Resistor_SMD:R_1206_3216Metric_Pad1.30x1.75mm_HandSolder
Changed lines of the file:
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@@
 			)
 		)
-		(property "Footprint" "Resistor_SMD:R_0805_2012Metric"
+		(property "Footprint" "Resistor_SMD:R_1206_3216Metric_Pad1.30x1.75mm_HandSolder"
 			(at 296.418 180.34 90)
 			(effects
@@
 			)
 		)
-		(property "Footprint" "Connector_Dsub:DSUB-15_Socket_Vertical_P2.77x2.84mm_MountingHoles"
+		(property "Footprint" "TE_DSUB:5787683 15 Pin Female Vertical"
 			(at 215.9 46.99 0)
 			(effects
@@
 			)
 		)
-		(property "Footprint" "Resistor_SMD:R_0805_2012Metric"
+		(property "Footprint" "Resistor_SMD:R_1206_3216Metric_Pad1.30x1.75mm_HandSolder"
 			(at 281.178 180.34 90)
 			(effects
@@
 			)
 		)
-		(property "Footprint" "Resistor_SMD:R_0805_2012Metric"
+		(property "Footprint" "Resistor_SMD:R_1206_3216Metric_Pad1.30x1.75mm_HandSolder"
 			(at 288.798 180.34 90)
 			(effects
@@
 			)
 		)
-		(property "Footprint" "Resistor_SMD:R_0805_2012Metric"
+		(property "Footprint" "Resistor_SMD:R_1206_3216Metric_Pad1.30x1.75mm_HandSolder"
 			(at 311.658 180.34 90)
 			(effects
@@
 			)
 		)
-		(property "Footprint" "Fuse:Fuse_0805_2012Metric"
+		(property "Footprint" "fuse_holder:FUSE_3568"
 			(at 119.38 175.26 0)
 			(effects
@@
 			)
 		)
-		(property "Footprint" "Resistor_SMD:R_0805_2012Metric"
+		(property "Footprint" "Resistor_SMD:R_1206_3216Metric_Pad1.30x1.75mm_HandSolder"
 			(at 304.038 180.34 90)
 			(effects
